Commit message: 1.1.1
- 실린더로 슬레이브 로봇 대체하기. 상수로 슬레이브 로봇 절대위치 받기
- 시뮬레이션 런치파일 만들기

File: mobile_robot_sim/urdf/slave_cylinder.urdf (robot description, URDF)
Before this commit: robot simple_box, 1 links, 0 joints
Links:
- removed link my_box
- added link slave_cylinder, mass 1.0; collision cylinder length=0.2 radius=0.075; visual cylinder length=0.2 radius=0.075
